Commit message: cleaning up the packages into extra_packages

File: ommp_description/urdf/arms/costum_arm/costum_arm.transmissions.xacro (robot description, xacro)
@@ -4,9 +4,9 @@
       <type>transmission_interface/SimpleTransmission</type>
       <joint name="joint_0">
-        <hardwareInterface>hardware_interface/EffortJointInterface</hardwareInterface>
+        <hardwareInterface>hardware_interface/PositionJointInterface</hardwareInterface>
       </joint>
       <actuator name="motor_joint_0">
         <mechanicalReduction>1</mechanicalReduction>
-	<hardwareInterface>hardware_interface/EffortJointInterface</hardwareInterface>
+	<hardwareInterface>hardware_interface/PositionJointInterface</hardwareInterface>
       </actuator>
     </transmission>
@@ -14,9 +14,9 @@
       <type>transmission_interface/SimpleTransmission</type>
       <joint name="joint_1">
-        <hardwareInterface>hardware_interface/EffortJointInterface</hardwareInterface>
+        <hardwareInterface>hardware_interface/PositionJointInterface</hardwareInterface>
       </joint>
       <actuator name="motor_joint_1">
         <mechanicalReduction>1</mechanicalReduction>
-	<hardwareInterface>hardware_interface/EffortJointInterface</hardwareInterface>
+	<hardwareInterface>hardware_interface/PositionJointInterface</hardwareInterface>
       </actuator>
     </transmission>
@@ -24,9 +24,9 @@
       <type>transmission_interface/SimpleTransmission</type>
       <joint name="joint_2">
-        <hardwareInterface>hardware_interface/EffortJointInterface</hardwareInterface>
+        <hardwareInterface>hardware_interface/PositionJointInterface</hardwareInterface>
       </joint>
       <actuator name="motor_joint_2">
         <mechanicalReduction>1</mechanicalReduction>
-	<hardwareInterface>hardware_interface/EffortJointInterface</hardwareInterface>
+	<hardwareInterface>hardware_interface/PositionJointInterface</hardwareInterface>
       </actuator>
     </transmission>
@@ -34,9 +34,9 @@
       <type>transmission_interface/SimpleTransmission</type>
       <joint name="joint_3">
-        <hardwareInterface>hardware_interface/EffortJointInterface</hardwareInterface>
+        <hardwareInterface>hardware_interface/PositionJointInterface</hardwareInterface>
       </joint>
       <actuator name="motor_joint_3">
         <mechanicalReduction>1</mechanicalReduction>
-	<hardwareInterface>hardware_interface/EffortJointInterface</hardwareInterface>
+	<hardwareInterface>hardware_interface/PositionJointInterface</hardwareInterface>
       </actuator>
     </transmission>
@@ -44,9 +44,9 @@
       <type>transmission_interface/SimpleTransmission</type>
       <joint name="joint_4">
-        <hardwareInterface>hardware_interface/EffortJointInterface</hardwareInterface>
+        <hardwareInterface>hardware_interface/PositionJointInterface</hardwareInterface>
       </joint>
       <actuator name="motor_joint_4">
         <mechanicalReduction>1</mechanicalReduction>
-	<hardwareInterface>hardware_interface/EffortJointInterface</hardwareInterface>
+	<hardwareInterface>hardware_interface/PositionJointInterface</hardwareInterface>
       </actuator>
     </transmission>
@@ -54,9 +54,9 @@
       <type>transmission_interface/SimpleTransmission</type>
       <joint name="joint_5">
-        <hardwareInterface>hardware_interface/EffortJointInterface</hardwareInterface>
+        <hardwareInterface>hardware_interface/PositionJointInterface</hardwareInterface>
       </joint>
       <actuator name="motor_joint_5">
         <mechanicalReduction>1</mechanicalReduction>
-	<hardwareInterface>hardware_interface/EffortJointInterface</hardwareInterface>
+	<hardwareInterface>hardware_interface/PositionJointInterface</hardwareInterface>
       </actuator>
     </transmission>

File: ommp_description/urdf/arms/costum_arm/costum_arm.urdf.xacro (robot description, xacro)
@@ -111,5 +111,5 @@
   <xacro:arm_joint joint_name="joint_5" parent="link_4" child = "link_5"
                type = "revolute"
-               origin_xyz = "-0.006 0 0.026"
+               origin_xyz = "0 0 0.026"
                origin_rpy = "0 0 0"
                axis_xyz = "0 0 1"

File: ommp_description/urdf/bases/lynxbot_base/lynxbot_bases.urdf.xacro (robot description, xacro)
@@ -15,5 +15,5 @@
        <origin xyz="0 0 0" rpy="0 0 0"/>
        <mass value="100"/>
-       <inertia ixx="0.5"  ixy="0"  ixz="0" iyy="0.5" iyz="0" izz="0.5" />
+       <inertia ixx="0.05"  ixy="0"  ixz="0" iyy="0.05" iyz="0" izz="0.05" />
      </inertial>
       <collision name='collision'>

File: ommp_description/urdf/robots/ommp_sim/ommp_sim.urdf.xacro (robot description, xacro)
@@ -1,6 +1,6 @@
 <?xml version='1.0'?>
-<robot name="lynx_rover" xmlns:xacro="http://www.ros.org/wiki/xacro">
+<robot name="ommp_sim" xmlns:xacro="http://www.ros.org/wiki/xacro">
   <!-- Common design Properties-->
-  <xacro:include filename="$(find ommp_description)/urdf/robots/lynxbot/common_properties.urdf.xacro" />
+  <xacro:include filename="$(find ommp_description)/urdf/robots/ommp_sim/common_properties.urdf.xacro" />
   <!-- Include Sensors macros -->
     <!--ydlidar -->
@@ -22,5 +22,5 @@
   <xacro:if value="$(arg sim)">
       <!-- General -->
-      <xacro:include filename="$(find ommp_description)/urdf/robots/lynxbot/lynx_rover.gazebo.xacro" />
+      <xacro:include filename="$(find ommp_description)/urdf/robots/ommp_sim/ommp_sim.gazebo.xacro" />
   </xacro:if>
   <!-- All the bases of the robot -->

File: ommp_description/urdf/sensors/kinect/kinect.urdf.xacro (robot description, xacro)
@@ -8,4 +8,5 @@
                        frame_name="camera_depth_optical_frame"/>
   </xacro:if>
+  	<!-- remove if Kinect isn't moving -->
     <xacro:include filename="$(find ommp_description)/urdf/sensors/kinect/kinect.transmissions.xacro" />
 	<!-- Parameterised in part by the values in kinect_properties.urdf.xacro -->

File: ommp_description/urdf/wheels/costum_wheel/costum_wheel.urdf.xacro (robot description, xacro)
@@ -27,5 +27,5 @@
         <origin xyz="0 0 0" rpy="0 0 0"/>
         <mass value="10"/>
-        <inertia ixx="0.15"  ixy="0"  ixz="0" iyy="0.15" iyz="0" izz="0.15" />
+        <inertia ixx="0.005"  ixy="0"  ixz="0" iyy="0.005" iyz="0" izz="0.005" />
       </inertial>
     </link>
