Commit message: Pre Organized

File: ommp_description/urdf/arms/costum_arm/costum_arm.urdf.xacro (robot description, xacro)
@@ -58,6 +58,6 @@
                axis_xyz = "0 1 0"
                axis_rpy = "0 0 0"
-	       lower_limit = "-0.8"
-               upper_limit = "2"/>
+	       lower_limit = "-1"
+               upper_limit = "1.57"/>
   <xacro:arm_link link_name="link_2" length="0.142" radius="0.01"
               origin_xyz="0 0 0.071"
@@ -72,6 +72,6 @@
                axis_xyz = "0 1 0"
                axis_rpy = "0 0 0"
-               lower_limit = "0.0"
-               upper_limit = "1.57"/>
+               lower_limit = "1.05"
+               upper_limit = "2.09"/>
   <xacro:arm_link link_name="link_3" length="0.02" radius="0.01"
               origin_xyz="0 0 0.01"

File: ommp_description/urdf/robots/ommp_real/common_properties.urdf.xacro (robot description, xacro)
@@ -58,5 +58,5 @@
   <xacro:property name="cam_pz" value="0.039" />
   <xacro:property name="cam_or" value="0.0" />
-  <xacro:property name="cam_op" value="0.0" />
+  <xacro:property name="cam_op" value="0.54" />
   <xacro:property name="cam_oy" value="0.0" />
   <!-- Arm -->

Commit message: Pre Organized

File: ommp_description/urdf/arms/costum_arm/costum_arm.urdf.xacro (robot description, xacro)
@@ -58,6 +58,6 @@
                axis_xyz = "0 1 0"
                axis_rpy = "0 0 0"
-	       lower_limit = "-0.8"
-               upper_limit = "2"/>
+	       lower_limit = "-1.57"
+               upper_limit = "2.57"/>
   <xacro:arm_link link_name="link_2" length="0.142" radius="0.01"
               origin_xyz="0 0 0.071"
@@ -73,5 +73,5 @@
                axis_rpy = "0 0 0"
                lower_limit = "0.0"
-               upper_limit = "1.57"/>
+               upper_limit = "3.14"/>
   <xacro:arm_link link_name="link_3" length="0.02" radius="0.01"
               origin_xyz="0 0 0.01"

File: ommp_description/urdf/robots/ommp_real/common_properties.urdf.xacro (robot description, xacro)
@@ -50,14 +50,15 @@
   <xacro:property name="lidar_parent" value="chassis" />
   <xacro:property name="lidar_joint_origin">
-    <origin xyz="0.026 0.0 0.047" rpy="0 0 0" /> <!-- height 0.67 or lower --> <!-- exprimental start base 15.5 -> -0.4 + 3-->
+    <origin xyz="0.026 0.0 0.058" rpy="0 0 3.098" /> <!-- height 0.67 or lower --> <!-- exprimental start base 15.5 -> -0.4 + 3-->
   </xacro:property>
   <!-- kinect base-->
   <xacro:property name="kinect_parent" value="kinect_base2" />
-  <xacro:property name="cam_px" value="0.02" />
+  <xacro:property name="cam_px" value="-0.02" />
   <xacro:property name="cam_py" value="0.0" />
-  <xacro:property name="cam_pz" value="0.039" />
+  <xacro:property name="cam_pz" value="0.095" /><!--0.35--> <!--0.095-->
   <xacro:property name="cam_or" value="0.0" />
-  <xacro:property name="cam_op" value="0.0" />
-  <xacro:property name="cam_oy" value="0.0" />
+  <!--xacro:property name="cam_op" value="0.0" /-->
+  <xacro:property name="cam_op" value="0.541" /> <!--0.541-->
+  <xacro:property name="cam_oy" value="0.02" />
   <!-- Arm -->
   <xacro:property name="arm_joint_origin">

Commit message: Working 1

File: ommp_description/urdf/arms/costum_arm/costum_arm.urdf.xacro (robot description, xacro)
@@ -14,4 +14,5 @@
 <xacro:property name="m_4" value="0.4" />
 <xacro:property name="m_5" value="0.4" />
+<!--Macro of the arm with the help of Link Joint Macros-->
 <xacro:macro name="costum_arm" params="parent">
   <joint name="arm_joint" type="fixed">
@@ -58,6 +59,6 @@
                axis_xyz = "0 1 0"
                axis_rpy = "0 0 0"
-	       lower_limit = "-1"
-               upper_limit = "1.57"/>
+	       lower_limit = "-1.57"
+               upper_limit = "2.35"/>
   <xacro:arm_link link_name="link_2" length="0.142" radius="0.01"
               origin_xyz="0 0 0.071"
@@ -72,6 +73,6 @@
                axis_xyz = "0 1 0"
                axis_rpy = "0 0 0"
-               lower_limit = "1.05"
-               upper_limit = "2.09"/>
+               lower_limit = "0.0"
+               upper_limit = "2.61"/>
   <xacro:arm_link link_name="link_3" length="0.02" radius="0.01"
               origin_xyz="0 0 0.01"

File: ommp_description/urdf/grippers/costum_gripper/costum_gripper.gazebo.xacro (robot description, xacro)
@@ -8,6 +8,6 @@
   <gazebo reference="finger1">
     <material>Gazebo/Black</material>
-    <mu1>30</mu1>
-    <mu2>30</mu2>
+    <mu1>300</mu1>
+    <mu2>300</mu2>
     <kd>1.0</kd>
     <kp>1000000.0</kp>
@@ -15,26 +15,8 @@
   <gazebo reference="finger2">
     <material>Gazebo/Black</material>
-    <mu1>30</mu1>
-    <mu2>30</mu2>
+    <mu1>300</mu1>
+    <mu2>300</mu2>
     <kd>1.0</kd>
     <kp>1000000.0</kp>
   </gazebo>
-  <!-- grasp plugin -->
-  <gazebo>
-    <plugin name="gazebo_grasp_fix" filename="libgazebo_grasp_fix.so">
-      <arm>
-        <arm_name>costum_arm</arm_name>
-        <palm_link>ee_base</palm_link>
-        <gripper_link>finger1</gripper_link>
-        <gripper_link>finger2</gripper_link>
-      </arm>
-      <forces_angle_tolerance>100</forces_angle_tolerance>
-      <update_rate>4</update_rate>
-      <grip_count_threshold>4</grip_count_threshold>
-      <max_grip_count>8</max_grip_count>
-      <release_tolerance>0.003</release_tolerance>
-      <disable_collisions_on_attach>true</disable_collisions_on_attach>
-      <contact_topic>__default_topic__</contact_topic>
-    </plugin>
-  </gazebo>
 </robot>

File: ommp_description/urdf/grippers/costum_gripper/costum_gripper.urdf.xacro (robot description, xacro)
@@ -5,21 +5,21 @@
       <!-- Gazebo gripper -->
       <xacro:include filename="$(find ommp_description)/urdf/grippers/costum_gripper/costum_gripper.gazebo.xacro" />
-      <xacro:include filename="$(find ommp_description)/urdf/grippers/costum_gripper/costum_gripper_effort.transmissions.xacro" />
+      <!--USE EFFORT IN SIM-->
+      <xacro:include filename="$(find ommp_description)/urdf/grippers/costum_gripper/costum_gripper_position.transmissions.xacro" />
   </xacro:if>
   <xacro:unless value="$(arg sim)">
+      <!--USE POS IN REAL-->
       <xacro:include filename="$(find ommp_description)/urdf/grippers/costum_gripper/costum_gripper_position.transmissions.xacro" />
   </xacro:unless>
-<xacro:property name="m_ee" value="0.1" />
+<xacro:property name="m_ee" value="0.01" />
 <xacro:property name="m_f1" value="0.01" />
 <xacro:property name="m_f2" value="0.01" />
 <xacro:macro name="costum_ee" params="parent">
-  <xacro:ee_joint joint_name="joint_ee_base" parent="${parent}" child = "ee_base"
+  <xacro:ee_base_joint joint_name="joint_ee_base" parent="${parent}" child = "ee_base"
                type = "fixed"
                origin_xyz = "0 0 0.006"
                origin_rpy = "0 0 0"
                axis_xyz = "0 0 1"
-               axis_rpy = "0 0 0"
-         lower_limit = "0"
-               upper_limit = "0"/>
+               axis_rpy = "0 0 0" />
   <xacro:ee_link link_name="ee_base" size_x="0.012" size_y="0.004" size_z="0.05"
               origin_xyz="0 0 0.004"

File: ommp_description/urdf/macros/inertia_macros.urdf.xacro (robot description, xacro)
@@ -37,5 +37,15 @@
     </inertial>
   </xacro:macro>
-  <xacro:macro name="cylinder_inertial1" params="radius length mass *origin">
+  <xacro:macro name="box_inertial2" params="x y z m *origin">
+    <inertial>
+      <mass value="${m}" />
+      <xacro:insert_block name="origin" />
+      <inertia  ixx="0.1" ixy = "0" ixz = "0"
+                  iyy="0.1" iyz = "0"
+                  izz="0.1" />
+    </inertial>
+  </xacro:macro>
+  <!--NOT USE THE FORMULLA -> 0.0001-->
+  <!--xacro:macro name="cylinder_inertial" params="radius length mass *origin">
     <inertial>
       <mass value="${mass}" />
@@ -45,4 +55,4 @@
         izz="${0.5 * mass * radius * radius}" />
     </inertial>
-  </xacro:macro>
+  </xacro:macro-->
 </robot>

File: ommp_description/urdf/macros/link_joint_macro.urdf.xacro (robot description, xacro)
@@ -54,5 +54,5 @@
       <collision>
         <geometry>
-          <box size="${size_x*0.5} ${size_y*0.5} ${size_z*0.5}"/>
+          <box size="${size_x*0.9} ${size_y*0.9} ${size_z*0.9}"/>
         </geometry>
         <origin xyz="${origin_xyz}" rpy="${origin_rpy}"/>
@@ -72,3 +72,12 @@
   </joint>
   </xacro:macro>
+  <xacro:macro name="ee_base_joint" params="joint_name type parent child
+    origin_xyz origin_rpy axis_xyz axis_rpy ">
+    <joint type="${type}" name="${joint_name}">
+    <origin xyz="${origin_xyz}" rpy="${origin_rpy}"/>
+    <child link="${child}"/>
+    <parent link="${parent}"/>
+    <axis xyz="${axis_xyz}" rpy="${axis_rpy}"/>
+  </joint>
+  </xacro:macro>
 </robot>

File: ommp_description/urdf/robots/ommp_real/ommp_real.urdf.xacro (robot description, xacro)
@@ -10,5 +10,5 @@
   <!--xacro:include filename="$(find ommp_description)/urdf/sensors/imu/imu.urdf.xacro" /-->
     <!-- kinect -->
-  <xacro:include filename="$(find ommp_description)/urdf/sensors/kinect/kinect.urdf.xacro" />
+  <xacro:include filename="$(find ommp_description)/urdf/sensors/kinect/kinect_real.urdf.xacro" />
   <!-- Include Bases-->
   <xacro:include filename="$(find ommp_description)/urdf/bases/lynxbot_base/lynxbot_bases.urdf.xacro" />

File: ommp_description/urdf/robots/ommp_sim/common_properties.urdf.xacro (robot description, xacro)
@@ -3,5 +3,5 @@
   <!-- Include or Not Gazebo Files-->
   <xacro:arg name="sim" default="true"/>
-  <xacro:arg name="gaz" default="true"/>
+  <xacro:property name="gz" default="true"/>
   <!-- PI Value -->
   <xacro:property name="M_PI" value="3.141592653" />
@@ -23,5 +23,5 @@
   </xacro:property>
   <xacro:property name="upper_base_joint_origin">
-    <origin xyz="0.05 0.0 0.1275" rpy="0 0 0" />
+    <origin xyz="0.05 0.0 0.0875" rpy="0 0 0" />
   </xacro:property>
   <xacro:property name="kinect_base1_size">
@@ -38,5 +38,5 @@
   </xacro:property>
   <!-- imu-->
-  <xacro:property name="imu_parent" value="chassis" />
+  <!--xacro:property name="imu_parent" value="chassis" />
   <xacro:property name="imu_size">
     <box size = "0.01 0.01 0.01"/>
@@ -44,21 +44,19 @@
   <xacro:property name="imu_joint_origin">
     <origin xyz="-0.1 0.0 0.0575" rpy="0 0 0" />
-  </xacro:property>
+  </xacro:property-->
   <!-- lidar base-->
   <xacro:property name="lidar_parent" value="chassis" />
   <xacro:property name="lidar_joint_origin">
-    <origin xyz="0.0 0.0 0.0575" rpy="0 0 0" />
+    <origin xyz="0.0 0.0 0.0315" rpy="0 0 0" />
   </xacro:property>
   <!-- kinect base-->
   <xacro:property name="kinect_parent" value="kinect_base2" />
-  <xacro:property name="cam_px" value="0.03" />
-  <xacro:property name="cam_py" value="0.0" />
-  <xacro:property name="cam_pz" value="0.055" />
-  <xacro:property name="cam_or" value="0.0" />
-  <xacro:property name="cam_op" value="0.0" />
-  <xacro:property name="cam_oy" value="0.0" />
+  <xacro:property name="kinect_joint_origin">
+    <origin xyz="0.03 0.0 0.055" rpy="0 0 0" />
+  </xacro:property>
+  <xacro:property name="cam_py" value="0" />
   <!-- Arm -->
   <xacro:property name="arm_joint_origin">
-    <origin xyz="0.079 0.0 0.02" rpy="0 0 0" />
+    <origin xyz="0.11 0.0 0.02" rpy="0 0 0" />
   </xacro:property>
   <xacro:property name="arm_parent" value="upper_base" />

File: ommp_description/urdf/robots/ommp_sim/ommp_sim.gazebo.xacro (robot description, xacro)
@@ -24,3 +24,31 @@
     </plugin>
   </gazebo-->
+  <!-- grasp plugin -->
+  <gazebo>
+    <plugin name="gazebo_grasp_fix" filename="libgazebo_grasp_fix.so">
+      <arm>
+        <arm_name>arm</arm_name>
+        <palm_link>finger1</palm_link>
+        <gripper_link>finger1</gripper_link>
+        <gripper_link>finger2</gripper_link>
+      </arm>
+      <forces_angle_tolerance>50</forces_angle_tolerance>
+      <update_rate>8</update_rate>
+      <grip_count_threshold>8</grip_count_threshold>
+      <max_grip_count>8</max_grip_count>
+      <release_tolerance>0.01</release_tolerance>
+      <disable_collisions_on_attach>true</disable_collisions_on_attach>
+      <contact_topic>__default_topic__</contact_topic>
+    </plugin>
+  </gazebo>
+  <!--gazebo>
+    <plugin name="omni_steering" filename="libgazebo_ros_planar_move.so">
+      <commandTopic>diff_velocity_controller/cmd_vel</commandTopic>
+      <odometryTopic>diff_velocity_controller/odom</odometryTopic>
+      <odometryFrame>odom</odometryFrame>
+      <odometryRate>50.0</odometryRate>
+      <robotBaseFrame>robot_footprint</robotBaseFrame>
+      <publishTF>true</publishTF>
+    </plugin>
+  </gazebo-->
 </robot>

File: ommp_description/urdf/robots/ommp_sim/ommp_sim.urdf.xacro (robot description, xacro)
@@ -1,15 +1,18 @@
 <?xml version='1.0'?>
 <robot name="ommp_sim" xmlns:xacro="http://www.ros.org/wiki/xacro">
+  <!--INCLUDE MACROS-->
   <!-- Common design Properties-->
   <xacro:include filename="$(find ommp_description)/urdf/robots/ommp_sim/common_properties.urdf.xacro" />
   <!-- Include Sensors macros -->
-    <!--ydlidar -->
+  <!---->
+  <!--ydlidar -->
   <xacro:include filename="$(find ommp_description)/urdf/sensors/ydlidar/ydlidar.urdf.xacro" />
-    <!--imu -->
-  <xacro:include filename="$(find ommp_description)/urdf/sensors/imu/imu.urdf.xacro" />
-    <!-- kinect -->
+  <!--imu -->
+  <!--xacro:include filename="$(find ommp_description)/urdf/sensors/imu/imu.urdf.xacro" /-->
+  <!-- kinect -->
   <xacro:include filename="$(find ommp_description)/urdf/sensors/kinect/kinect_sim.urdf.xacro" />
+  <!---->
   <!-- Include Bases-->
-  <xacro:include filename="$(find ommp_description)/urdf/bases/lynxbot_base/lynxbot_bases.urdf.xacro" />
+  <xacro:include filename="$(find ommp_description)/urdf/bases/ommp_base/ommp_bases.urdf.xacro" />
   <!-- Wheel Macro-->
   <xacro:include filename="$(find ommp_description)/urdf/wheels/costum_wheel/costum_wheel.urdf.xacro" />
@@ -21,20 +24,21 @@
   <xacro:include filename="$(find ommp_description)/urdf/grippers/costum_gripper/costum_gripper.urdf.xacro" />
   <xacro:if value="$(arg sim)">
-      <!-- General -->
-      <xacro:include filename="$(find ommp_description)/urdf/robots/ommp_sim/ommp_sim.gazebo.xacro" />
+    <!-- General e.g ros_control_plugin, gazebo grasp -->
+    <xacro:include filename="$(find ommp_description)/urdf/robots/ommp_sim/ommp_sim.gazebo.xacro" />
   </xacro:if>
+  <!--INSTANTIATE MACROS-->
   <!-- All the bases of the robot -->
   <xacro:lynxbot_bases />
   <!-- Instanciate the 4 wheels of the robot -->
-  <xacro:costum_wheel prefix="front_left" parent="chassis" gz="true">
+  <xacro:costum_wheel prefix="front_left" parent="chassis" gz="${gz}">
     <origin xyz="${wheel_offset_x} ${wheel_offset_y} ${wheel_offset_z}" rpy="0 0 0"/>
   </xacro:costum_wheel>
-  <xacro:costum_wheel prefix="front_right" parent="chassis" gz="true">
+  <xacro:costum_wheel prefix="front_right" parent="chassis" gz="${gz}">
     <origin xyz="${wheel_offset_x} -${wheel_offset_y} ${wheel_offset_z}" rpy="0 0 0"/>
   </xacro:costum_wheel>
-  <xacro:costum_wheel prefix="back_left" parent="chassis" gz="true">
+  <xacro:costum_wheel prefix="back_left" parent="chassis" gz="${gz}">
     <origin xyz="-${wheel_offset_x} ${wheel_offset_y} ${wheel_offset_z}" rpy="0 0 0"/>
   </xacro:costum_wheel>
-  <xacro:costum_wheel prefix="back_right" parent="chassis" gz="true">
+  <xacro:costum_wheel prefix="back_right" parent="chassis" gz="${gz}">
     <origin xyz="-${wheel_offset_x} -${wheel_offset_y} ${wheel_offset_z}" rpy="0 0 0"/>
   </xacro:costum_wheel>
@@ -43,5 +47,5 @@
   <xacro:sensor_kinect parent="${kinect_parent}" />
   <xacro:sensor_laser parent="chassis" />
-  <xacro:imu_sensor parent="chassis" />
+  <!--xacro:imu_sensor parent="chassis" /-->
   <!-- connect arm -->
   <xacro:costum_arm parent="${arm_parent}" />

File: ommp_description/urdf/sensors/kinect/kinect.gazebo.xacro (robot description, xacro)
@@ -1,4 +1,4 @@
 <?xml version="1.0"?>
-<robot name="kinect_gazebo" xmlns:xacro="http://www.ros.org/wiki/xacro">
+<robot xmlns:xacro="http://www.ros.org/wiki/xacro">
   <!-- Microsoft Kinect / ASUS Xtion PRO Live for simulation -->
   <xacro:macro name="kinect_gazebo_sensor" params="link_name camera_name frame_name">

File: ommp_description/urdf/sensors/kinect/kinect_sim.urdf.xacro (robot description, xacro)
@@ -5,5 +5,5 @@
       <xacro:include filename="$(find ommp_description)/urdf/sensors/kinect/kinect.gazebo.xacro" />
       <!-- Instantiate it -->
-      <xacro:kinect_gazebo_sensor link_name="camera_depth_frame" camera_name="camera"
+      <xacro:kinect_gazebo_sensor link_name="camera_depth_frame" camera_name="my_camera"
                        frame_name="camera_depth_optical_frame"/>
   </xacro:if>
@@ -13,5 +13,5 @@
 	<xacro:macro name="sensor_kinect" params="parent">
     <joint name="camera_rgb_joint" type="revolute">
-      <origin xyz="${cam_px} ${cam_py} ${cam_pz}" rpy="${cam_or} ${cam_op} ${cam_oy}"/>
+      <xacro:insert_block name="kinect_joint_origin" />
       <parent link="${parent}" />
       <child link="camera_rgb_frame" />
@@ -21,9 +21,4 @@
       <safety_controller k_velocity="10" k_position="15" soft_lower_limit="-1.57" soft_upper_limit="1.57" />
     </joint>
-    <!--joint name="camera_rgb_joint" type="fixed">
-      <origin xyz="0.031 ${-cam_py} 0.016" rpy="0 0 0"/>
-      <parent link="kinect_dummy"/>
-      <child link="camera_rgb_frame" />
-    </joint-->
     <link name="camera_rgb_frame">
       <inertial>

File: ommp_description/urdf/wheels/costum_wheel/costum_wheel.urdf.xacro (robot description, xacro)
@@ -8,6 +8,7 @@
       <xacro:insert_block name="origin" />
       <axis xyz="0 1 0" rpy="0 0 0" />
-      <limit effort="10000" velocity="1000"/>
-      <joint_properties damping="20.0" friction="10.0"/>
+      <limit effort="100" velocity="100"/>
+      <joint_properties damping="0.0" friction="0.0"/>
+      <!--joint_properties-->
     </joint>
     <link name="${prefix}_wheel_link">
@@ -30,5 +31,5 @@
         <origin xyz="0 0 0" rpy="0 0 0"/>
         <mass value="10"/>
-        <inertia ixx="0.005"  ixy="0"  ixz="0" iyy="0.005" iyz="0" izz="0.005" />
+        <inertia ixx="0.05"  ixy="0"  ixz="0" iyy="0.05" iyz="0" izz="0.05" />
       </inertial>
     </link>
@@ -45,11 +46,11 @@
     <xacro:if value="${gz}">
       <gazebo reference="${prefix}_wheel_link">
-      <!--mu1 value="1.0"/>
-      <mu2 value="1.0"/>
-      <kp value="10000000.0" />
-      <kd value="1.0" />
-      <fdir1 value="1 0 0"/>
-          <turnGravityOff>false</turnGravityOff-->
-      <material>Gazebo/Blue</material>
+        <mu1 value="1.0"/>
+        <mu2 value="1.0"/>
+        <kp value="10000000.0" />
+        <kd value="1.0" />
+        <fdir1 value="1 0 0"/>
+            <turnGravityOff>false</turnGravityOff>
+        <material>Gazebo/Blue</material>
       </gazebo>
     </xacro:if>
