Commit message: start on jetson

File: ommp_description/urdf/grippers/costum_gripper/costum_gripper.urdf.xacro (robot description, xacro)
@@ -2,9 +2,12 @@
 <robot xmlns:xacro="http://www.ros.org/wiki/xacro">
  <xacro:include filename="$(find ommp_description)/urdf/macros/link_joint_macro.urdf.xacro" />
- <xacro:include filename="$(find ommp_description)/urdf/grippers/costum_gripper/costum_gripper.transmissions.xacro" />
   <xacro:if value="$(arg sim)">
       <!-- Gazebo gripper -->
       <xacro:include filename="$(find ommp_description)/urdf/grippers/costum_gripper/costum_gripper.gazebo.xacro" />
+      <xacro:include filename="$(find ommp_description)/urdf/grippers/costum_gripper/costum_gripper_effort.transmissions.xacro" />
   </xacro:if>
+  <xacro:unless value="$(arg sim)">
+      <xacro:include filename="$(find ommp_description)/urdf/grippers/costum_gripper/costum_gripper_position.transmissions.xacro" />
+  </xacro:unless>
 <xacro:property name="m_ee" value="0.1" />
 <xacro:property name="m_f1" value="0.01" />

File: ommp_description/urdf/robots/ommp_real/common_properties.urdf.xacro (robot description, xacro)
@@ -2,6 +2,6 @@
 <robot xmlns:xacro="http://www.ros.org/wiki/xacro">
   <!-- Include or Not Gazebo Files-->
-  <xacro:arg name="sim" default="true"/>
-  <xacro:arg name="gaz" default="true"/>
+  <xacro:arg name="sim" default="false"/>
+  <xacro:arg name="gaz" default="false"/>
   <!-- PI Value -->
   <xacro:property name="M_PI" value="3.141592653" />
@@ -9,33 +9,34 @@
   <!--chassis-->
   <xacro:property name="base_size">
-    <box size = "0.25 0.2 0.06"/>
+    <box size = "0.318 0.2 0.008"/>
   </xacro:property>
   <!-- wheels-->
   <xacro:property name="wheel_size">
-    <cylinder length = "0.065" radius="0.055"/>
+    <cylinder length = "0.06" radius="0.05"/>
   </xacro:property>
-  <xacro:property name="wheel_offset_x" value="0.0975" />
-  <xacro:property name="wheel_offset_y" value="0.14" />
-  <xacro:property name="wheel_offset_z" value="-0.015" />
+  <xacro:property name="wheel_offset_x" value="0.14" />
+  <xacro:property name="wheel_offset_y" value="0.135" /> <!--+0.005-->
+  <xacro:property name="wheel_offset_z" value="-0.019" />
   <!--Robot bases-->
   <xacro:property name="upper_base_size">
-    <box size = "0.3 0.15 0.02"/>
+    <box size = "0.318 0.2 0.008"/>
   </xacro:property>
   <xacro:property name="upper_base_joint_origin">
-    <origin xyz="0.05 0.0 0.1275" rpy="0 0 0" />
+    <origin xyz="0.0 0.0 0.108" rpy="0 0 0" />
   </xacro:property>
   <xacro:property name="kinect_base1_size">
-    <box size = "0.01 0.03 0.38"/>
+    <box size = "0.01 0.03 0.4"/>
+  </xacro:property>
+  <xacro:property name="kinect_base1_joint_origin">
+    <origin xyz="-0.154 0.0 0.204" rpy="0 0 0" />
   </xacro:property>
   <xacro:property name="kinect_base2_size">
-    <box size = "0.07 0.07 0.02"/>
-  </xacro:property>
-  <xacro:property name="kinect_base1_joint_origin">
-    <origin xyz="-0.14 0.0 0.2" rpy="0 0 0" />
+    <box size = "0.1 0.07 0.008"/>
   </xacro:property>
   <xacro:property name="kinect_base2_joint_origin">
-    <origin xyz="0.035 0.0 0.19" rpy="0 0 0" />
+    <origin xyz="0.055 0.0 0.196" rpy="0 0 0" />
   </xacro:property>
   <!-- imu-->
+  <!--
   <xacro:property name="imu_parent" value="chassis" />
   <xacro:property name="imu_size">
@@ -45,14 +46,15 @@
     <origin xyz="-0.1 0.0 0.0575" rpy="0 0 0" />
   </xacro:property>
+  -->
   <!-- lidar base-->
   <xacro:property name="lidar_parent" value="chassis" />
   <xacro:property name="lidar_joint_origin">
-    <origin xyz="0.0 0.0 0.0575" rpy="0 0 0" />
+    <origin xyz="0.026 0.0 0.047" rpy="0 0 0" /> <!-- height 0.67 or lower --> <!-- exprimental start base 15.5 -> -0.4 + 3-->
   </xacro:property>
   <!-- kinect base-->
   <xacro:property name="kinect_parent" value="kinect_base2" />
-  <xacro:property name="cam_px" value="0.03" />
+  <xacro:property name="cam_px" value="0.02" />
   <xacro:property name="cam_py" value="0.0" />
-  <xacro:property name="cam_pz" value="0.055" />
+  <xacro:property name="cam_pz" value="0.039" />
   <xacro:property name="cam_or" value="0.0" />
   <xacro:property name="cam_op" value="0.0" />
@@ -60,5 +62,5 @@
   <!-- Arm -->
   <xacro:property name="arm_joint_origin">
-    <origin xyz="0.079 0.0 0.02" rpy="0 0 0" />
+    <origin xyz="0.119 0.0 0.024" rpy="0 0 0" />
   </xacro:property>
   <xacro:property name="arm_parent" value="upper_base" />

File: ommp_description/urdf/robots/ommp_real/ommp_real.urdf.xacro (robot description, xacro)
@@ -1,13 +1,14 @@
 <?xml version='1.0'?>
-<robot name="ommp_sim" xmlns:xacro="http://www.ros.org/wiki/xacro">
+<robot name="ommp_real" xmlns:xacro="http://www.ros.org/wiki/xacro">
+  <arg name="sim" default="true"/>
   <!-- Common design Properties-->
-  <xacro:include filename="$(find ommp_description)/urdf/robots/ommp_sim/common_properties.urdf.xacro" />
+  <xacro:include filename="$(find ommp_description)/urdf/robots/ommp_real/common_properties.urdf.xacro" />
   <!-- Include Sensors macros -->
     <!--ydlidar -->
   <xacro:include filename="$(find ommp_description)/urdf/sensors/ydlidar/ydlidar.urdf.xacro" />
     <!--imu -->
-  <xacro:include filename="$(find ommp_description)/urdf/sensors/imu/imu.urdf.xacro" />
+  <!--xacro:include filename="$(find ommp_description)/urdf/sensors/imu/imu.urdf.xacro" /-->
     <!-- kinect -->
-  <xacro:include filename="$(find ommp_description)/urdf/sensors/kinect/kinect_sim.urdf.xacro" />
+  <xacro:include filename="$(find ommp_description)/urdf/sensors/kinect/kinect.urdf.xacro" />
   <!-- Include Bases-->
   <xacro:include filename="$(find ommp_description)/urdf/bases/lynxbot_base/lynxbot_bases.urdf.xacro" />
@@ -20,21 +21,17 @@
   <!-- Include costum Gripper -->
   <xacro:include filename="$(find ommp_description)/urdf/grippers/costum_gripper/costum_gripper.urdf.xacro" />
-  <xacro:if value="$(arg sim)">
-      <!-- General -->
-      <xacro:include filename="$(find ommp_description)/urdf/robots/ommp_sim/ommp_sim.gazebo.xacro" />
-  </xacro:if>
   <!-- All the bases of the robot -->
   <xacro:lynxbot_bases />
   <!-- Instanciate the 4 wheels of the robot -->
-  <xacro:costum_wheel prefix="front_left" parent="chassis" gz="true">
+  <xacro:costum_wheel prefix="front_left" parent="chassis" gz="false">
     <origin xyz="${wheel_offset_x} ${wheel_offset_y} ${wheel_offset_z}" rpy="0 0 0"/>
   </xacro:costum_wheel>
-  <xacro:costum_wheel prefix="front_right" parent="chassis" gz="true">
+  <xacro:costum_wheel prefix="front_right" parent="chassis" gz="false">
     <origin xyz="${wheel_offset_x} -${wheel_offset_y} ${wheel_offset_z}" rpy="0 0 0"/>
   </xacro:costum_wheel>
-  <xacro:costum_wheel prefix="back_left" parent="chassis" gz="true">
+  <xacro:costum_wheel prefix="back_left" parent="chassis" gz="false">
     <origin xyz="-${wheel_offset_x} ${wheel_offset_y} ${wheel_offset_z}" rpy="0 0 0"/>
   </xacro:costum_wheel>
-  <xacro:costum_wheel prefix="back_right" parent="chassis" gz="true">
+  <xacro:costum_wheel prefix="back_right" parent="chassis" gz="false">
     <origin xyz="-${wheel_offset_x} -${wheel_offset_y} ${wheel_offset_z}" rpy="0 0 0"/>
   </xacro:costum_wheel>
@@ -43,5 +40,5 @@
   <xacro:sensor_kinect parent="${kinect_parent}" />
   <xacro:sensor_laser parent="chassis" />
-  <xacro:imu_sensor parent="chassis" />
+  <!--xacro:imu_sensor parent="chassis" /-->
   <!-- connect arm -->
   <xacro:costum_arm parent="${arm_parent}" />

File: ommp_description/urdf/sensors/kinect/kinect_sim.urdf.xacro (robot description, xacro)
@@ -12,17 +12,8 @@
 	<!-- Parameterised in part by the values in kinect_properties.urdf.xacro -->
 	<xacro:macro name="sensor_kinect" params="parent">
-    <link name="kinect_dummy">
-      <inertial>
-        <mass value="0.001" />
-        <origin xyz="0 0 0" />
-        <inertia ixx="0.0001" ixy="0.0" ixz="0.0"
-                 iyy="0.0001" iyz="0.0"
-                 izz="0.0001" />
-      </inertial>
-    </link>
-    <joint name="camera_dummy_joint" type="revolute">
+    <joint name="camera_rgb_joint" type="revolute">
       <origin xyz="${cam_px} ${cam_py} ${cam_pz}" rpy="${cam_or} ${cam_op} ${cam_oy}"/>
       <parent link="${parent}" />
-      <child link="kinect_dummy" />
+      <child link="camera_rgb_frame" />
       <axis xyz="0 1 0" rpy="0 0 0" />
       <dynamics damping="0.0" friction="0.0"/>
@@ -30,9 +21,9 @@
       <safety_controller k_velocity="10" k_position="15" soft_lower_limit="-1.57" soft_upper_limit="1.57" />
     </joint>
-    <joint name="camera_rgb_joint" type="fixed">
-      <origin xyz="0.03 ${-cam_py} 0.016" rpy="0 0 0"/>
+    <!--joint name="camera_rgb_joint" type="fixed">
+      <origin xyz="0.031 ${-cam_py} 0.016" rpy="0 0 0"/>
       <parent link="kinect_dummy"/>
       <child link="camera_rgb_frame" />
-    </joint>
+    </joint-->
     <link name="camera_rgb_frame">
       <inertial>

File: ommp_description/urdf/wheels/costum_wheel/costum_wheel.urdf.xacro (robot description, xacro)
@@ -17,4 +17,7 @@
           <xacro:insert_block name="wheel_size" />
         </geometry>
+        <material name="blue">
+          <color rgba="1 0 0 1"/>
+        </material>
       </visual>
       <collision>
