Commit message: Real bringup working in master

File: ommp_packages/ommp_description/urdf/robots/ommp_real/common_properties.urdf.xacro (robot description, xacro)
@@ -50,14 +50,15 @@
   <xacro:property name="lidar_parent" value="chassis" />
   <xacro:property name="lidar_joint_origin">
-    <origin xyz="0.026 0.0 0.047" rpy="0 0 0" /> <!-- height 0.67 or lower --> <!-- exprimental start base 15.5 -> -0.4 + 3-->
+    <origin xyz="0.026 0.0 0.058" rpy="0 0 3.098" /> <!-- height 0.67 or lower --> <!-- exprimental start base 15.5 -> -0.4 + 3-->
   </xacro:property>
   <!-- kinect base-->
   <xacro:property name="kinect_parent" value="kinect_base2" />
-  <xacro:property name="cam_px" value="0.02" />
+  <xacro:property name="cam_px" value="-0.02" />
   <xacro:property name="cam_py" value="0.0" />
-  <xacro:property name="cam_pz" value="0.039" />
+  <xacro:property name="cam_pz" value="0.095" /><!--0.35--> <!--0.095-->
   <xacro:property name="cam_or" value="0.0" />
-  <xacro:property name="cam_op" value="0.54" />
-  <xacro:property name="cam_oy" value="0.0" />
+  <!--xacro:property name="cam_op" value="0.0" /-->
+  <xacro:property name="cam_op" value="0.541" /> <!--0.541-->
+  <xacro:property name="cam_oy" value="0.02" />
   <!-- Arm -->
   <xacro:property name="arm_joint_origin">

File: ommp_packages/ommp_description/urdf/robots/ommp_real/ommp_real.urdf.xacro (robot description, xacro)
@@ -1,5 +1,5 @@
 <?xml version='1.0'?>
 <robot name="ommp_real" xmlns:xacro="http://www.ros.org/wiki/xacro">
-  <arg name="sim" default="true"/>
+  <arg name="sim" default="false"/>
   <!-- Common design Properties-->
   <xacro:include filename="$(find ommp_description)/urdf/robots/ommp_real/common_properties.urdf.xacro" />
@@ -8,9 +8,9 @@
   <xacro:include filename="$(find ommp_description)/urdf/sensors/ydlidar/ydlidar.urdf.xacro" />
     <!--imu -->
-  <!--xacro:include filename="$(find ommp_description)/urdf/sensors/imu/imu.urdf.xacro" /-->
+  <xacro:include filename="$(find ommp_description)/urdf/sensors/imu/imu.urdf.xacro" />
     <!-- kinect -->
   <xacro:include filename="$(find ommp_description)/urdf/sensors/kinect/kinect_real.urdf.xacro" />
   <!-- Include Bases-->
-  <xacro:include filename="$(find ommp_description)/urdf/bases/lynxbot_base/lynxbot_bases.urdf.xacro" />
+  <xacro:include filename="$(find ommp_description)/urdf/bases/ommp_base_real/ommp_bases.urdf.xacro" />
   <!-- Wheel Macro-->
   <xacro:include filename="$(find ommp_description)/urdf/wheels/costum_wheel/costum_wheel.urdf.xacro" />
@@ -22,5 +22,5 @@
   <xacro:include filename="$(find ommp_description)/urdf/grippers/costum_gripper/costum_gripper.urdf.xacro" />
   <!-- All the bases of the robot -->
-  <xacro:lynxbot_bases />
+  <xacro:ommp_bases />
   <!-- Instanciate the 4 wheels of the robot -->
   <xacro:costum_wheel prefix="front_left" parent="chassis" gz="false">
@@ -40,5 +40,5 @@
   <xacro:sensor_kinect parent="${kinect_parent}" />
   <xacro:sensor_laser parent="chassis" />
-  <!--xacro:imu_sensor parent="chassis" /-->
+  <xacro:imu_sensor parent="chassis" />
   <!-- connect arm -->
   <xacro:costum_arm parent="${arm_parent}" />
