Commit message: STABLE

File: ommp_packages/ommp_description/urdf/macros/inertia_macros.urdf.xacro (robot description, xacro)
@@ -1,5 +1,5 @@
 <?xml version="1.0" ?>
 <robot xmlns:xacro="http://www.ros.org/wiki/xacro">
-  <!--xacro:macro name="cylinder_inertial" params="radius length mass *origin">
+  <xacro:macro name="cylinder_inertial" params="radius length mass *origin">
     <inertial>
       <mass value="${mass}" />
@@ -10,49 +10,21 @@
     </inertial>
   </xacro:macro>
-  <xacro:macro name="box_inertial" params="x y z m *origin">
-    <inertial>
-      <mass value="${m}" />
-      <xacro:insert_block name="origin" />
-      <inertia  ixx="${m*(y*y+z*z)/12}" ixy = "0" ixz = "0"
-                  iyy="${m*(x*x+z*z)/12}" iyz = "0"
-                  izz="${m*(x*x+z*z)/12}" />
-    </inertial>
-  </xacro:macro-->
-  <xacro:macro name="cylinder_inertial" params="radius length mass *origin">
+  <xacro:macro name="box_inertial" params="x y z mass *origin">
     <inertial>
       <mass value="${mass}" />
       <xacro:insert_block name="origin" />
-      <inertia  ixx="0.0001" ixy = "0" ixz = "0"
-                  iyy="0.0001" iyz = "0"
-                  izz="0.0001" />
+      <inertia ixx="${0.0833333 * mass * (y * y + z * z)}" ixy="0.0" ixz="0.0"
+        iyy="${0.0833333 * mass * (x * x + z * z)}" iyz="0.0"
+        izz="${0.0833333 * mass * (x * x + z * z)}" />
     </inertial>
   </xacro:macro>
-  <xacro:macro name="box_inertial" params="x y z m *origin">
+  <xacro:macro name="inertial_dummy" params="*origin">
     <inertial>
-      <mass value="${m}" />
+      <mass value="0.01" />
       <xacro:insert_block name="origin" />
-      <inertia  ixx="0.0001" ixy = "0" ixz = "0"
-                  iyy="0.0001" iyz = "0"
-                  izz="0.0001" />
+      <inertia ixx="0.0001" ixy="0.0" ixz="0.0"
+        iyy="0.0001" iyz="0.0"
+        izz="0.0001" />
     </inertial>
   </xacro:macro>
-  <xacro:macro name="box_inertial2" params="x y z m *origin">
-    <inertial>
-      <mass value="${m}" />
-      <xacro:insert_block name="origin" />
-      <inertia  ixx="0.1" ixy = "0" ixz = "0"
-                  iyy="0.1" iyz = "0"
-                  izz="0.1" />
-    </inertial>
-  </xacro:macro>
-  <!--NOT USE THE FORMULLA -> 0.0001-->
-  <!--xacro:macro name="cylinder_inertial" params="radius length mass *origin">
-    <inertial>
-      <mass value="${mass}" />
-      <xacro:insert_block name="origin" />
-      <inertia ixx="${0.0833333 * mass * (3 * radius * radius + length * length)}" ixy="0.0" ixz="0.0"
-        iyy="${0.0833333 * mass * (3 * radius * radius + length * length)}" iyz="0.0"
-        izz="${0.5 * mass * radius * radius}" />
-    </inertial>
-  </xacro:macro-->
 </robot>

File: ommp_packages/ommp_description/urdf/robots/ommp_real/ommp_real.urdf.xacro (robot description, xacro)
@@ -3,5 +3,5 @@
   <arg name="sim" default="false"/>
   <!-- Common design Properties-->
-  <xacro:include filename="$(find ommp_description)/urdf/robots/ommp_real/common_properties.urdf.xacro" />
+  <xacro:include filename="$(find ommp_description)/urdf/robots/ommp_real/configuration.urdf.xacro" />
   <!-- Include Sensors macros -->
     <!--ydlidar -->
@@ -18,7 +18,7 @@
   <xacro:include filename="$(find ommp_description)/urdf/macros/inertia_macros.urdf.xacro" />
   <!-- Include costum Arm -->
-  <xacro:include filename="$(find ommp_description)/urdf/arms/costum_arm/costum_arm.urdf.xacro" />
+  <xacro:include filename="$(find ommp_description)/urdf/arms/generic_arm/generic_arm.urdf.xacro" />
   <!-- Include costum Gripper -->
-  <xacro:include filename="$(find ommp_description)/urdf/grippers/costum_gripper/costum_gripper.urdf.xacro" />
+  <xacro:include filename="$(find ommp_description)/urdf/grippers/generic_gripper/generic_gripper.urdf.xacro" />
   <!-- All the bases of the robot -->
   <xacro:ommp_bases />
@@ -41,7 +41,20 @@
   <xacro:sensor_laser parent="chassis" />
   <xacro:imu_sensor parent="chassis" />
+  <!-- Instanciate the Generic Arm macros -->
   <!-- connect arm -->
-  <xacro:costum_arm parent="${arm_parent}" />
+  <xacro:generic_arm
+    prefix=""
+    parent="${generic_arm_parent}"
+    transmission_hw_interface="${transmission_hw_interface}"
+    safety_limits="${safety_limits}"
+    safety_pos_margin="${safety_pos_margin}"
+    safety_k_position="${safety_k_position}"/>
   <!-- connect gripper-->
-  <xacro:costum_ee parent="${ee_parent}" />
+  <xacro:generic_gripper
+    prefix=""
+    parent="${generic_gripper_parent}"
+    transmission_hw_interface="${transmission_hw_interface}"
+    safety_limits="${safety_limits}"
+    safety_pos_margin="${safety_pos_margin}"
+    safety_k_position="${safety_k_position}"/>
 </robot>

File: ommp_packages/ommp_description/urdf/robots/ommp_sim/ommp_sim.urdf.xacro (robot description, xacro)
@@ -3,5 +3,5 @@
   <!--INCLUDE MACROS-->
   <!-- Common design Properties-->
-  <xacro:include filename="$(find ommp_description)/urdf/robots/ommp_sim/common_properties.urdf.xacro" />
+  <xacro:include filename="$(find ommp_description)/urdf/robots/ommp_sim/configuration.urdf.xacro" />
   <!-- Include Sensors macros -->
   <!---->
@@ -19,8 +19,8 @@
   <!-- Incude Inertia macros -->
   <xacro:include filename="$(find ommp_description)/urdf/macros/inertia_macros.urdf.xacro" />
-  <!-- Include costum Arm -->
-  <xacro:include filename="$(find ommp_description)/urdf/arms/costum_arm/costum_arm.urdf.xacro" />
-  <!-- Include costum Gripper -->
-  <xacro:include filename="$(find ommp_description)/urdf/grippers/costum_gripper/costum_gripper.urdf.xacro" />
+  <!-- Include Generic Arm -->
+  <xacro:include filename="$(find ommp_description)/urdf/arms/generic_arm/generic_arm.urdf.xacro" />
+  <!-- Include Generic Gripper -->
+  <xacro:include filename="$(find ommp_description)/urdf/grippers/generic_gripper/generic_gripper.urdf.xacro" />
   <xacro:if value="$(arg sim)">
     <!-- General e.g ros_control_plugin, gazebo grasp -->
@@ -48,7 +48,20 @@
   <xacro:sensor_laser parent="chassis" />
   <xacro:imu_sensor parent="chassis" />
+  <!-- Instanciate the Generic Arm macros -->
   <!-- connect arm -->
-  <xacro:costum_arm parent="${arm_parent}" />
+  <xacro:generic_arm
+    prefix=""
+    parent="${generic_arm_parent}"
+    transmission_hw_interface="${transmission_hw_interface}"
+    safety_limits="${safety_limits}"
+    safety_pos_margin="${safety_pos_margin}"
+    safety_k_position="${safety_k_position}"/>
   <!-- connect gripper-->
-  <xacro:costum_ee parent="${ee_parent}" />
+  <xacro:generic_gripper
+    prefix=""
+    parent="${generic_gripper_parent}"
+    transmission_hw_interface="${transmission_hw_interface}"
+    safety_limits="${safety_limits}"
+    safety_pos_margin="${safety_pos_margin}"
+    safety_k_position="${safety_k_position}"/>
 </robot>
